File: HackPadCase.kicad_pcb (KiCad board)
At the start: 2 copper layers, 81.5 x 41.6 mm, 15 parts, among them SW1 SW_Push, SW2 SW_Push, SW3 SW_Push, SW4 SW_Push, SW5 SW_Push, SW6 SW_Push, SW7 RotaryEncoder_Switch, U1 Seeed Studio XIAO SAMD21

Commit message: upd8
Parts:
- added G***: LOGO, hp:Sachh, B.Cu at (190.2, 71.1)
- D1, D2, D3, D4, D5, D6: moved to B.Cu
- U1: moved to F.Cu
- moved D5 61.2 mm to (140.0, 65.9), turned to -90 degrees
- moved D6 58.4 mm to (140.0, 86.0), turned to -90 degrees
- moved D4 51.8 mm to (140.0, 83.5)
- moved G*** 38.7 mm to (160.5, 98.9)
- moved D3 34.2 mm to (159.2, 74.7)
- moved D2 24.2 mm to (159.4, 95.0)
- moved D1 22.8 mm to (159.3, 84.9)
- moved U1 0.92 mm to (190.4, 91.0), turned to -90 degrees
Routing:
- net Column 1: track 102.1 -> 158.4 mm
- net Net-(D4-A): track 70.3 -> 15.9 mm
- net Net-(U1-PB08_A6_D6_TX): track 48.7 -> 6.44 mm
- net Net-(D3-A): track 44.2 -> 7.51 mm
- net Net-(U1-PA9_A5_D5_SCL): track 38.7 -> 8.90 mm
- net Net-(D2-A): track 53.6 -> 28.5 mm
- net Net-(D1-A): track 56.7 -> 32.5 mm
- net Column 2: track 130.6 -> 108.1 mm
- net Net-(SW7-PadC): track 6.51 -> 27.5 mm
- net Net-(D6-A): track 28.2 -> 44.1 mm
- net Column 3: track 69.7 -> 83.8 mm
- net Net-(D5-A): track 33.3 -> 37.8 mm
